File: board2/DCMotorController/DCMotorController.kicad_pcb (KiCad board)
At the start: 4 copper layers, 85 x 90 mm, 97 parts, among them J1 Conn_01x02, J2 Conn_01x02, M1_S1 Conn_01x03_Female, M1_S2 Conn_01x03_Female, Q1 Q_NMOS_GDS, Q2 Q_NMOS_GDS, Q3 Q_NMOS_GDS, Q4 Q_NMOS_GDS, Q5 Q_NMOS_GDS, Q6 Q_NMOS_GDS, Q7 Q_NMOS_GDS, Q8 Q_NMOS_GDS, U1 INA180A1, U10 TPS54360DDA, U2 IR2103, U3 IR2103, U4 ESP32-WROOM-32D, U9 DS18B20

Commit message: v2 ordering
Parts:
- C1, C10, C15, C18, C2, C33, C34, C35, C5, C8: footprint Capacitor_SMD:C_0603_1608Metric -> PCM_Capacitor_SMD_AKL:C_0603_1608Metric
- C11, C12, C7, C9: footprint PCM_Capacitor_SMD_AKL:C_1206_3216Metric_Pad1.42x1.75mm_HandSolder -> PCM_Capacitor_SMD_Handsoldering_AKL:C_1206_3216Metric
- C13, C31, C32: footprint Capacitor_SMD:C_1206_3216Metric -> PCM_Capacitor_SMD_Handsoldering_AKL:C_1206_3216Metric
- C4, C6: footprint PCM_Capacitor_SMD_AKL:C_0805_2012Metric_Pad1.15x1.40mm_HandSolder -> PCM_Capacitor_SMD_Handsoldering_AKL:C_0805_2012Metric
- U4: footprint RF_Module:ESP32-WROOM-32 -> esp_no_wifi:ESP32-WROOM-32_no_wifi
- U9: footprint Connector_PinHeader_1.00mm:PinHeader_1x03_P1.00mm_Vertical -> Package_TO_SOT_THT:TO-92_Inline
- moved C17 3.89 mm to (97.0, 72.0), turned to 180 degrees
- moved J2 1.40 mm to (112.6, 21.8)
- moved U9 1.08 mm to (94.5, 28.5), turned to 90 degrees
- moved TP3V3_0V1 0.19 mm to (99.6, 93.9)
- renumbered Rvoltage1 to R11, Rvoltage2 to R19, Rvoltage3 to R20, Rvoltage4 to R24
Connections:
- net Net-(D1-K) renamed M+
- net Net-(D4-K) renamed M-
- C18 pad 1: BAT- -> GND
Routing:
- net M-: track 159.8 -> 60.3 mm, vias 2 -> 60
- net GND: track 302.0 -> 203.6 mm, vias 5 -> 104
- net VIN: track 123.6 -> 26.2 mm, vias 1 -> 92
- net M+: track 119.0 -> 52.8 mm, vias 0 -> 55
- net BAT-: track 32.4 -> 17.9 mm
- net Net-(U2-VB): track 15.2 -> 25.0 mm
- net VMosfet: track 56.3 -> 61.7 mm
- net Net-(U3-VB): track 15.4 -> 18.5 mm
- net 3_3V: track 246.9 -> 244.0 mm
- net Temp: track 116.4 -> 114.6 mm
- net Net-(D6-A): track 63.1 -> 64.6 mm
- net Net-(D3-A): track 12.4 -> 11.6 mm
- net Net-(D5-A): track 64.4 -> 63.8 mm
- net Net-(D5-K): track 10.7 -> 10.1 mm
- net (no net): vias 0 -> 1
- added copper zone on B.Cu, net BAT-
- added copper zone on F.Cu, net BAT-
- added copper zone on In1.Cu, net BAT-
- added copper zone on In2.Cu, net BAT-
- added copper zone on B.Cu, net M+
- added copper zone on F.Cu, net M+
- added copper zone on In1.Cu, net M+
- added copper zone on In2.Cu, net M+
- added copper zone on B.Cu, net M-
- added copper zone on F.Cu, net M-
- added copper zone on In1.Cu, net M-
- added copper zone on In2.Cu, net M-
- added copper zone on B.Cu, net VIN
- added copper zone on F.Cu, net VIN
- added copper zone on In1.Cu, net VIN
- added copper zone on In2.Cu, net VIN
Other:
- outline, holes or cut-outs redrawn
- board text added: "DCBrushed 2.0 max 60V 60A"
