File: board2/DCMotorController/DCMotorController.kicad_sch (KiCad schematic)
At the start: 97 parts, among them J1 Conn_01x02, J2 Conn_01x02, M1_S1 Conn_01x03_Female, M1_S2 Conn_01x03_Female, Q1 Q_NMOS_GDS, Q2 Q_NMOS_GDS, Q3 Q_NMOS_GDS, Q4 Q_NMOS_GDS, Q5 Q_NMOS_GDS, Q6 Q_NMOS_GDS, Q7 Q_NMOS_GDS, Q8 Q_NMOS_GDS, U1 INA180A1, U10 TPS54360DDA, U2 IR2103, U3 IR2103, U4 ESP32-WROOM-32D, U9 DS18B20

Commit message: v2 ordering
Parts:
- C1, C10, C15, C18, C2, C33, C34, C35, C5, C8: footprint Capacitor_SMD:C_0603_1608Metric -> PCM_Capacitor_SMD_AKL:C_0603_1608Metric
- C11, C12, C7, C9: footprint PCM_Capacitor_SMD_AKL:C_1206_3216Metric_Pad1.42x1.75mm_HandSolder -> PCM_Capacitor_SMD_Handsoldering_AKL:C_1206_3216Metric
- C13, C31, C32: footprint Capacitor_SMD:C_1206_3216Metric -> PCM_Capacitor_SMD_Handsoldering_AKL:C_1206_3216Metric
- C4, C6: footprint PCM_Capacitor_SMD_AKL:C_0805_2012Metric_Pad1.15x1.40mm_HandSolder -> PCM_Capacitor_SMD_Handsoldering_AKL:C_0805_2012Metric
- GND_TX_RX1: symbol Connector:Conn_01x03_Male -> Connector_Generic:Conn_01x03
- M1_S1, M1_S2: symbol Connector:Conn_01x03_Female -> Connector_Generic:Conn_01x03
- R1: LCSC (none) -> C695947
- U4: footprint RF_Module:ESP32-WROOM-32 -> esp_no_wifi:ESP32-WROOM-32_no_wifi
- U9: footprint Connector_PinHeader_1.00mm:PinHeader_1x03_P1.00mm_Vertical -> Package_TO_SOT_THT:TO-92_Inline
- renumbered Rvoltage1 to R11, Rvoltage2 to R19, Rvoltage3 to R20, Rvoltage4 to R24
Connections:
- net BAT-: no longer C18.1
- net GND: now also C18.1
- net M+: now reaches C7.2, D1.1 (K), J2.1 (Pin_1), P1.3 (0V), Q3.3 (S), Q4.3 (S), Q7.2 (D), Q8.2 (D), TPVMos0V2.1, U3.6 (VS)
- net M-: now reaches C9.2, D4.1 (K), J2.2 (Pin_2), P2.3 (0V), Q1.3 (S), Q2.2 (D), Q5.3 (S), Q6.2 (D), TPVMos0V3.1, U2.6 (VS)
- no-connect marks 17 -> 22
